Commit message: Add motor characteristics' ROS Param

File: sample/xacro/position_pid_servo.xacro (robot description, xacro)
@@ -81,5 +81,5 @@
     <origin xyz="1.0 0 0.5" rpy="0 -1.57 0"/>
     <axis xyz="0 1 0"/>
-    <limit effort="1000.0" lower="-3.14" upper="3.14" velocity="1000.0"/>
+    <limit effort="10000.0" lower="-3.14" upper="3.14" velocity="10000.0"/>
     <dynamics damping="0" friction="0"/>
   </joint>
@@ -116,5 +116,5 @@
     <origin xyz="1.0 0 0" rpy="0 -1.57 0"/>
     <axis xyz="0 1 0"/>
-    <limit effort="1000.0" lower="-3.14" upper="3.14" velocity="1000.0"/>
+    <limit effort="10000.0" lower="-3.14" upper="3.14" velocity="10000.0"/>
     <dynamics damping="0" friction="0"/>
   </joint>
@@ -151,5 +151,5 @@
     <origin xyz="1.0 0 0" rpy="0 -1.57 0"/>
     <axis xyz="0 1 0"/>
-    <limit effort="1000.0" lower="-3.14" upper="3.14" velocity="1000.0"/>
+    <limit effort="10000.0" lower="-3.14" upper="3.14" velocity="10000.0"/>
     <dynamics damping="0" friction="0"/>
   </joint>
