Commit message: Add default mode

File: sample/xacro/test_wheel.xacro (robot description, xacro)
@@ -40,4 +40,7 @@
           <hardwareInterface>hardware_interface/EffortJointInterface</hardwareInterface>
         </xacro:if>
+        <xacro:if value="${gazebo_control_mode=='position'}">
+          <hardwareInterface>hardware_interface/PositionJointInterface</hardwareInterface>
+        </xacro:if>
         <xacro:if value="${gazebo_control_mode=='velocity'}">
           <hardwareInterface>hardware_interface/VelocityJointInterface</hardwareInterface>
@@ -47,4 +50,11 @@
     </transmission>
   </xacro:macro>
+<!--   <link name="world"/>
+  <joint name="world_joint" type="fixed">
+    <parent link="world"/>
+    <child  link="right_pad2"/>
+    <origin xyz="0 0 0" rpy="0 0 0"/>
+    <axis xyz="0 0 1"/>
+  </joint> -->
   <link name="right_pad2">
     <visual>
